Commit message: Even more octorotor_description fixes

File: hector_octorotor_description/urdf/octorotor.gazebo.xacro (robot description, xacro)
@@ -2,4 +2,4 @@
 <robot name="octorotor" xmlns:xacro="http://www.ros.org/wiki/xacro">
     <xacro:include filename="$(find hector_octorotor_description)/urdf/octorotor.urdf.xacro" />
-    <xacro:include filename="$(find hector_quadrotor_gazebo)/urdf/quadrotor_plugins.gazebo.xacro" />
+    <xacro:include filename="$(find hector_octorotor_gazebo)/urdf/octorotor_plugins.gazebo.xacro" />
 </robot>

File: hector_octorotor_description/urdf/octorotor_base.urdf.xacro (robot description, xacro)
@@ -14,5 +14,5 @@
         <origin xyz="0 0 0" rpy="0 0 0" />
         <geometry>
-          <mesh filename="package://hector_quadrotor_description/meshes/octorotor/octorotor_base.dae"/>
+          <mesh filename="package://hector_octorotor_description/meshes/octorotor/octorotor_base.dae"/>
         </geometry>
       </visual>
@@ -20,5 +20,5 @@
         <origin xyz="0 0 0" rpy="0 0 0" />
         <geometry>
-          <mesh filename="package://hector_quadrotor_description/meshes/quadrotor/quadrotor_base.stl"/>
+          <mesh filename="package://hector_octorotor_description/meshes/octorotor/quadrotor_base.stl"/>
           <!-- TODO: THIS SHOULD BE CHANGED AS WELL -->
         </geometry>
