Commit message: Final fixes for octorotor_base

File: hector_octorotor_description/urdf/octorotor_base.urdf.xacro (robot description, xacro)
@@ -30,5 +30,5 @@
 		    <origin xyz="0 0 0" rpy="0 0 0" />
 		    <geometry>
-		      <mesh filename="package://hector_octorotor_description/meshes/octorotor/quadrotor_base.stl"/>
+		      <mesh filename="package://hector_octorotor_description/meshes/octorotor/octorotor_base.stl"/>
 		      <!-- TODO: THIS SHOULD BE CHANGED AS WELL -->
 		    </geometry>
